File: _autosave-PCB-MIDI-THRU.sch (KiCad schematic (older format))
At the start: 61 parts, among them J1 Conn_02x05_Odd_Even, J2 Conn_01x02_Male, J3 Conn_01x02_Male, J4 Conn_01x02_Male, J5 Conn_01x02_Male, J6 Conn_01x02_Male, J7 Conn_01x02_Male, U1 L7805, U2 6N136, U3 74LS14

Commit message: v0.0.1 PCB SCHEM
Parts:
- added C9: C, Capacitor_THT:C_Disc_D4.3mm_W1.9mm_P5.00mm, symbol Device:C
Connections:
- net +5V: now also C9.1
- net GND: now also C9.2
- net at D1.1 (K), U1.1 (IN): now also C1.1, D2.1 (K)
Changed lines of the file:
@@
 $EndComp
 Wire Wire Line
-	1900 3700 2100 3700
+	1900 3700 2050 3700
 Wire Wire Line
 	2700 3700 2900 3700
@@
 	2200 3300 2050 3300
 Wire Wire Line
-	2050 3300 2050 3950
+	2050 3300 2050 3700
 Wire Wire Line
 	2700 4150 2400 4150
@@
 Text Notes 7500 6800 0    50   ~ 0
 MIDI THRU V0.0.1
+$Comp
+L Device:C C9
+U 1 1 60331913
+P 4150 4150
+F 0 "C9" H 4265 4196 50  0000 L CNN
+F 1 "C" H 4265 4105 50  0000 L CNN
+F 2 "Capacitor_THT:C_Disc_D4.3mm_W1.9mm_P5.00mm" H 4188 4000 50  0001 C CNN
+F 3 "~" H 4150 4150 50  0001 C CNN
+	1    4150 4150
+	1    0    0    -1
+$EndComp
+Wire Wire Line
+	4150 3650 4150 4000
+Wire Wire Line
+	3500 3650 4150 3650
+Connection ~ 3500 3650
+Wire Wire Line
+	3500 4650 4150 4650
+Wire Wire Line
+	4150 4650 4150 4300
+Connection ~ 3500 4650
+Connection ~ 2050 3700
+Wire Wire Line
+	2050 3700 2100 3700
+Wire Wire Line
+	2050 3700 2050 3950
 $EndSCHEMATC
