File: PCB-MIDI-THRU.kicad_pcb (KiCad board)
At the start: 2 copper layers, 61 parts, among them J1 Conn_02x05_Odd_Even, J2 Conn_01x02_Male, J3 Conn_01x02_Male, J4 Conn_01x02_Male, J5 Conn_01x02_Male, J6 Conn_01x02_Male, J7 Conn_01x02_Male, U1 L7805, U2 6N136, U3 74LS14

Commit message: v0.0.1 PCB SCHEM
Parts:
- added C9: 0.1uf, Capacitor_THT:C_Disc_D4.3mm_W1.9mm_P5.00mm, F.Cu at (186.6, 131.0)
- added H1: MountingHole_Pad, MountingHole:MountingHole_3.2mm_M3_DIN965_Pad, F.Cu at (236.0, 140.6)
- added H2: MountingHole_Pad, MountingHole:MountingHole_3.2mm_M3_DIN965_Pad, F.Cu at (109.7, 140.6)
- added H2: MountingHole_Pad, MountingHole:MountingHole_3.2mm_M3_DIN965_Pad, F.Cu at (162.5, 140.6)
- D12, D13, D14, D15, D16, D6: moved to B.Cu
- J2: value Conn_01x02_Male -> Midi In; moved to B.Cu
- J3: value Conn_01x02_Male -> Midi-Thru-1; moved to B.Cu
- J4: value Conn_01x02_Male -> Midi-Thru-2; moved to B.Cu
- J5: value Conn_01x02_Male -> Midi-Thru-3; moved to B.Cu
- J6: value Conn_01x02_Male -> Midi-Thru-4; moved to B.Cu
- J7: value Conn_01x02_Male -> Midi-Thru-5; moved to B.Cu
- moved D7 152.9 mm to (153.2, 158.0), turned to 90 degrees
- moved C4 125.7 mm to (153.2, 140.6)
- moved J3 123.2 mm to (150.7, 122.3)
- moved C2 121.0 mm to (104.2, 151.1), turned to 180 degrees
- moved R1 120.5 mm to (123.1, 160.8), turned to 180 degrees
- moved R13 114.8 mm to (143.0, 148.0), turned to 90 degrees
- moved D2 114.6 mm to (104.1, 135.6), turned to 270 degrees
- moved D8 113.4 mm to (178.2, 158.0), turned to 90 degrees
- moved D12 113.0 mm to (143.0, 122.5), turned to 90 degrees
- moved R18 112.1 mm to (147.6, 150.5), turned to 270 degrees
- moved D3 111.9 mm to (123.3, 156.3), turned to 180 degrees
- moved J2 109.7 mm to (108.9, 154.7), turned to 180 degrees
- moved U2 109.4 mm to (127.1, 152.1)
- moved R23 109.2 mm to (147.5, 137.8), turned to 270 degrees
- moved J1 109.0 mm to (94.1, 145.7)
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Connections:
- D1 pad 1: Net-(D1-Pad1) -> Net-(C1-Pad1)
- U1 pad 1: Net-(D1-Pad1) -> Net-(C1-Pad1)
Other:
- board outline added: 175 x 47 mm
- board text added: "CLAYTUNE MidiThru By TwinTurbo V0.0.1"
- board text added: "For Kate"
- board text added: "JLCJLCJLCJLC"
- board text added: "https://electronics.stackexchange.com/questions/281467/midi-activity-led"

Commit message: v0.0.1 PCB SCHEM b
Parts:
- D4: moved to B.Cu
- moved D4 2.88 mm to (94.4, 156.0), turned to 180 degrees
Changed lines of the file:
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@@
     (descr "Through hole IDC box header, 2x05, 2.54mm pitch, DIN 41651 / IEC 60603-13, double rows, https://docs.google.com/spreadsheets/d/16SsEcesNF15N3Lb4niX7dcUr-NY5_MFPQhobNuNppn4/edit#gid=0")
     (tags "Through hole vertical IDC box header THT 2x05 2.54mm double row")
-    (fp_text reference J1 (at 1.77 -12.02) (layer F.SilkS)
+    (fp_text reference J1 (at 7.23 -4.98) (layer F.SilkS)
       (effects (font (size 1 1) (thickness 0.15)))
     )
@@
     )
   )
-  (module LED_THT:LED_D5.0mm (layer F.Cu)
-    (at 91.61 156.58)
+  (module LED_THT:LED_D5.0mm (layer B.Cu)
+    (at 94.44 156.03 180)
     (descr "LED, diameter 5.0mm, 2 pins, http://cdn-reichelt.de/documents/datenblatt/A500/LL-504BC2E-009.pdf")
     (tags "LED diameter 5.0mm 2 pins")
-    (fp_text reference D4 (at 5.61 -2.53) (layer F.SilkS)
-      (effects (font (size 1 1) (thickness 0.15)))
-    )
-    (fp_text value POWER (at -2.77 0.18 90) (layer F.Fab)
-      (effects (font (size 1 1) (thickness 0.15)))
-    )
-    (fp_text user %R (at 1.25 0) (layer F.Fab)
-      (effects (font (size 0.8 0.8) (thickness 0.2)))
-    )
-    (fp_arc (start 1.27 0) (end -1.29 1.54483) (angle -148.9) (layer F.SilkS) (width 0.12))
-    (fp_arc (start 1.27 0) (end -1.29 -1.54483) (angle 148.9) (layer F.SilkS) (width 0.12))
-    (fp_arc (start 1.27 0) (end -1.23 -1.469694) (angle 299.1) (layer F.Fab) (width 0.1))
-    (fp_circle (center 1.27 0) (end 3.77 0) (layer F.Fab) (width 0.1))
-    (fp_circle (center 1.27 0) (end 3.77 0) (layer F.SilkS) (width 0.12))
-    (fp_line (start -1.23 -1.469694) (end -1.23 1.469694) (layer F.Fab) (width 0.1))
-    (fp_line (start -1.29 -1.545) (end -1.29 1.545) (layer F.SilkS) (width 0.12))
-    (fp_line (start -1.95 -3.25) (end -1.95 3.25) (layer F.CrtYd) (width 0.05))
-    (fp_line (start -1.95 3.25) (end 4.5 3.25) (layer F.CrtYd) (width 0.05))
-    (fp_line (start 4.5 3.25) (end 4.5 -3.25) (layer F.CrtYd) (width 0.05))
-    (fp_line (start 4.5 -3.25) (end -1.95 -3.25) (layer F.CrtYd) (width 0.05))
-    (pad 2 thru_hole circle (at 2.54 0) (size 1.8 1.8) (drill 0.9) (layers *.Cu *.Mask)
+    (fp_text reference D4 (at 5.61 2.53) (layer B.SilkS)
+      (effects (font (size 1 1) (thickness 0.15)) (justify mirror))
+    )
+    (fp_text value POWER (at -2.77 -0.18 270) (layer B.Fab)
+      (effects (font (size 1 1) (thickness 0.15)) (justify mirror))
+    )
+    (fp_text user %R (at 1.25 0) (layer B.Fab)
+      (effects (font (size 0.8 0.8) (thickness 0.2)) (justify mirror))
+    )
+    (fp_arc (start 1.27 0) (end -1.29 -1.54483) (angle 148.9) (layer B.SilkS) (width 0.12))
+    (fp_arc (start 1.27 0) (end -1.29 1.54483) (angle -148.9) (layer B.SilkS) (width 0.12))
+    (fp_arc (start 1.27 0) (end -1.23 1.469694) (angle -299.1) (layer B.Fab) (width 0.1))
+    (fp_circle (center 1.27 0) (end 3.77 0) (layer B.Fab) (width 0.1))
+    (fp_circle (center 1.27 0) (end 3.77 0) (layer B.SilkS) (width 0.12))
+    (fp_line (start -1.23 1.469694) (end -1.23 -1.469694) (layer B.Fab) (width 0.1))
+    (fp_line (start -1.29 1.545) (end -1.29 -1.545) (layer B.SilkS) (width 0.12))
+    (fp_line (start -1.95 3.25) (end -1.95 -3.25) (layer B.CrtYd) (width 0.05))
+    (fp_line (start -1.95 -3.25) (end 4.5 -3.25) (layer B.CrtYd) (width 0.05))
+    (fp_line (start 4.5 -3.25) (end 4.5 3.25) (layer B.CrtYd) (width 0.05))
+    (fp_line (start 4.5 3.25) (end -1.95 3.25) (layer B.CrtYd) (width 0.05))
+    (pad 2 thru_hole circle (at 2.54 0 180) (size 1.8 1.8) (drill 0.9) (layers *.Cu *.Mask)
       (net 13 "Net-(D4-Pad2)"))
-    (pad 1 thru_hole rect (at 0 0) (size 1.8 1.8) (drill 0.9) (layers *.Cu *.Mask)
+    (pad 1 thru_hole rect (at 0 0 180) (size 1.8 1.8) (drill 0.9) (layers *.Cu *.Mask)
       (net 1 GND))
     (model ${KISYS3DMOD}/LED_THT.3dshapes/LED_D5.0mm.wrl

Commit message: v0.0.1 Front
Parts:
- added G***: LOGO, AA-ROB-FULL:K6neg, B.Cu at (176.3, 140.7)
- added H1: MountingHole_Pad, MountingHole:MountingHole_3.2mm_M3_DIN965_Pad, F.Cu at (236.0, 128.6)
- added H2: MountingHole_Pad, MountingHole:MountingHole_3.2mm_M3_DIN965_Pad, F.Cu at (162.5, 152.6)
- D10, D11, D5, D7, D8, D9: value 1N4001 -> 1N4148
- J2: value Midi In -> Conn_01x02_Male
- J3: value Midi-Thru-1 -> Conn_01x02_Male
- J4: value Midi-Thru-2 -> Conn_01x02_Male
- J5: value Midi-Thru-3 -> Conn_01x02_Male
- J6: value Midi-Thru-4 -> Conn_01x02_Male
- J7: value Midi-Thru-5 -> Conn_01x02_Male
- moved H1 12.0 mm to (236.0, 152.6)
- moved H2 12.0 mm to (162.5, 128.6)

Commit message: v0.0.1 pcb routed
Parts:
- renumbered H2 to H1, H2 to H3, H1 to H4, H1 to H5
Routing:
- net +5V: track 0.00 -> 184.1 mm
- net Net-(R2-Pad1): track 0.00 -> 99.3 mm
- net Net-(D11-Pad1): track 0.00 -> 87.4 mm
- net Net-(R7-Pad1): track 0.00 -> 83.4 mm
- net Net-(D7-Pad1): track 0.00 -> 74.4 mm
- net Net-(D9-Pad1): track 0.00 -> 62.7 mm
- net Net-(D10-Pad1): track 0.00 -> 54.0 mm
- net Net-(D8-Pad1): track 0.00 -> 44.2 mm
- net Net-(D5-Pad1): track 0.00 -> 34.1 mm
- net Net-(J7-Pad2): track 0.00 -> 31.9 mm
- net Net-(J6-Pad2): track 0.00 -> 31.9 mm
- net Net-(J5-Pad2): track 0.00 -> 31.9 mm
- net Net-(J4-Pad2): track 0.00 -> 31.9 mm
- net Net-(J3-Pad2): track 0.00 -> 31.9 mm
- net Net-(J7-Pad1): track 0.00 -> 31.5 mm
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- added copper zone on B.Cu, net GND
- added copper zone on F.Cu, net GND
