File: PCB-MIDI-THRU.kicad_pcb (KiCad board)
At the start: 2 copper layers, 175 x 47 mm, 68 parts, among them J1 Conn_02x05_Odd_Even, J2 Conn_01x02_Male, J3 Conn_01x02_Male, J4 Conn_01x02_Male, J5 Conn_01x02_Male, J6 Conn_01x02_Male, J7 Conn_01x02_Male, U1 L7805, U2 6N136, U3 74LS14

Commit message: Fixed PCB up to v0.0.2
Parts:
- U2: value 6N136 -> 6N137
Connections:
- U2 pad 4: Net-(U2-Pad4) -> (no net)
- U2 pad 5: Net-(U2-Pad5) -> GND
Routing:
- net GND: track 0.00 -> 52.0 mm
Other:
- board text added: "CLAYTUNE MidiThru By TwinTurbo V0.0.2"
- board text added: "V0.0.2"
- board text removed: "CLAYTUNE MidiThru By TwinTurbo V0.0.1"
Changed lines of the file:
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@@
   (general
     (thickness 1.6)
-    (drawings 8)
-    (tracks 301)
+    (drawings 9)
+    (tracks 307)
     (zones 0)
     (modules 68)
-    (nets 44)
+    (nets 42)
   )
   (page A4)
@@
     (35 F.Paste user)
     (36 B.SilkS user hide)
-    (37 F.SilkS user hide)
+    (37 F.SilkS user)
     (38 B.Mask user)
     (39 F.Mask user)
@@
   (net 38 "Net-(R2-Pad1)")
   (net 39 "Net-(R7-Pad1)")
-  (net 40 "Net-(U2-Pad4)")
-  (net 41 "Net-(U2-Pad7)")
-  (net 42 "Net-(U2-Pad5)")
-  (net 43 "Net-(U2-Pad1)")
+  (net 40 "Net-(U2-Pad7)")
+  (net 41 "Net-(U2-Pad1)")
   (net_class Default "This is the default net class."
     (clearance 0.2)
@@
     (add_net "Net-(R7-Pad1)")
     (add_net "Net-(U2-Pad1)")
-    (add_net "Net-(U2-Pad4)")
-    (add_net "Net-(U2-Pad5)")
     (add_net "Net-(U2-Pad7)")
   )
@@
       (effects (font (size 1 1) (thickness 0.15)))
     )
-    (fp_text value 6N136 (at 3.81 9.95) (layer F.SilkS)
+    (fp_text value 6N137 (at 3.81 9.95) (layer F.SilkS)
       (effects (font (size 1 1) (thickness 0.15)))
     )
@@
     (pad 8 thru_hole oval (at 7.62 0) (size 1.6 1.6) (drill 0.8) (layers *.Cu *.Mask)
       (net 3 +5V))
-    (pad 4 thru_hole oval (at 0 7.62) (size 1.6 1.6) (drill 0.8) (layers *.Cu *.Mask)
-      (net 40 "Net-(U2-Pad4)"))
+    (pad 4 thru_hole oval (at 0 7.62) (size 1.6 1.6) (drill 0.8) (layers *.Cu *.Mask))
     (pad 7 thru_hole oval (at 7.62 2.54) (size 1.6 1.6) (drill 0.8) (layers *.Cu *.Mask)
-      (net 41 "Net-(U2-Pad7)"))
+      (net 40 "Net-(U2-Pad7)"))
     (pad 3 thru_hole oval (at 0 5.08) (size 1.6 1.6) (drill 0.8) (layers *.Cu *.Mask)
       (net 11 "Net-(D3-Pad2)"))
@@
       (net 12 "Net-(D3-Pad1)"))
     (pad 5 thru_hole oval (at 7.62 7.62) (size 1.6 1.6) (drill 0.8) (layers *.Cu *.Mask)
-      (net 42 "Net-(U2-Pad5)"))
+      (net 1 GND))
     (pad 1 thru_hole rect (at 0 0) (size 1.6 1.6) (drill 0.8) (layers *.Cu *.Mask)
-      (net 43 "Net-(U2-Pad1)"))
+      (net 41 "Net-(U2-Pad1)"))
     (model ${KISYS3DMOD}/Package_DIP.3dshapes/DIP-8_W7.62mm.wrl
       (at (xyz 0 0 0))
@@
     )
   )
+  (gr_text V0.0.2 (at 201.82 169.72) (layer F.SilkS)
+    (effects (font (size 1 1) (thickness 0.15)))
+  )
   (gr_text https://electronics.stackexchange.com/questions/281467/midi-activity-led (at 231.78 180.09) (layer F.Cu)
     (effects (font (size 1.5 1.5) (thickness 0.3)))
@@
     (effects (font (size 1.5 1.5) (thickness 0.3) italic))
   )
-  (gr_text "CLAYTUNE\nMidiThru\nBy TwinTurbo \nV0.0.1" (at 208.98 129.38 180) (layer F.SilkS)
+  (gr_text "CLAYTUNE\nMidiThru\nBy TwinTurbo \nV0.0.2" (at 208.98 129.38 180) (layer F.SilkS)
     (effects (font (size 1.5 1.5) (thickness 0.3) italic))
   )
@@
   (gr_line (start 257.6 117.1) (end 257.6 164.1) (layer Edge.Cuts) (width 0.05))
   (gr_line (start 82.6 164.1) (end 257.6 164.1) (layer Edge.Cuts) (width 0.05))
+  (segment (start 134.71 159.7) (end 131.4 163.01) (width 0.25) (layer F.Cu) (net 1))
+  (segment (start 131.4 163.01) (end 106.01 163.01) (width 0.25) (layer F.Cu) (net 1))
+  (segment (start 101.65 158.65) (end 101.65 151.14) (width 0.25) (layer F.Cu) (net 1))
+  (segment (start 106.01 163.01) (end 101.65 158.65) (width 0.25) (layer F.Cu) (net 1))
+  (segment (start 99.03 156.03) (end 101.65 158.65) (width 0.25) (layer F.Cu) (net 1))
+  (segment (start 94.44 156.03) (end 99.03 156.03) (width 0.25) (layer F.Cu) (net 1))
   (segment (start 115.32 140.96) (end 115.32 139.6822) (width 0.25) (layer B.Cu) (net 2))
   (segment (start 104.12 134.9773) (end 110.6151 134.9773) (width 0.25) (layer B.Cu) (net 2))

Commit message: PCB minus input LED
Parts:
- removed C3: 10UF, Capacitor_THT:CP_Radial_D5.0mm_P2.50mm
- removed D5: 1N4148, Diode_THT:D_A-405_P10.16mm_Horizontal
- removed D6: LED, LED_THT:LED_D5.0mm
- removed the G*** at (176.3, 140.7)
- removed R4, R7: LINK, Resistor_THT:R_Axial_DIN0207_L6.3mm_D2.5mm_P10.16mm_Horizontal
- removed R5: 4K7, Resistor_THT:R_Axial_DIN0207_L6.3mm_D2.5mm_P10.16mm_Horizontal
- removed R6: 470R, Resistor_THT:R_Axial_DIN0207_L6.3mm_D2.5mm_P10.16mm_Horizontal
- added G***: LOGO, AA-ROB-FULL:GF-X1FC, F.Cu at (126.1, 128.0)
- H1: value MountingHole_Pad -> H3
- H2: value MountingHole_Pad -> H2
- H3: value MountingHole_Pad -> H1
- H4: value MountingHole_Pad -> H4
- H5: value MountingHole_Pad -> H5
- U2: value 6N137 -> 6N136
- moved H1 54.1 mm to (109.7, 140.6)
- moved H3 54.1 mm to (162.5, 152.6)
- moved H2 24.0 mm to (162.5, 128.6)
Connections:
- H1 pad 1: (no net) -> GND
- H2 pad 1: (no net) -> GND
- H3 pad 1: (no net) -> GND
- H4 pad 1: (no net) -> GND
- H5 pad 1: (no net) -> GND
Routing:
- net GND: track 52.0 -> 3.42 mm
- net Net-(D5-Pad1): track 34.1 -> 0.00 mm
- net Net-(U3-Pad11): track 83.4 -> 66.3 mm
- net Net-(C3-Pad1): track 15.8 -> 0.00 mm
- net Net-(D6-Pad2): track 12.5 -> 0.00 mm
- net Net-(R2-Pad1): track 99.3 -> 99.8 mm, vias 0 -> 1

Commit message: PCB V0.0.3
Other:
- board text added: "CLAYTUNE MidiThru By TwinTurbo V0.0.3"
- board text removed: "CLAYTUNE MidiThru By TwinTurbo V0.0.2"

Commit message: DOC Version Number Update
Other:
- board text added: "V0.0.3"
- board text removed: "V0.0.2"
