File: Front/Panel.kicad_pcb (KiCad board)
At the start: 2 copper layers, 485.8 x 320.1 mm, 27 parts, among them SW9 RUNSTOP

Commit message: v0.0.1 Front
Parts:
- removed the +12V at (17.0, 33.8)
- removed -12V: LED -12, RobsFoots:FP-LED_D5.0mm
- removed the H1 at (459.2, -40.5)
- removed the H1 at (180.9, 152.0)
- removed the H1 at (137.9, 152.0)
- removed the H1 at (100.7, 215.2)
- removed the H1 at (82.7, 215.2)
- removed the H1 at (82.7, 22.2)
- removed the H1 at (40.9, 172.0)
- removed the H1 at (54.4, 109.0)
- removed the H1 at (100.7, 22.2)
- removed the H1 at (366.2, 152.5)
- removed the H1 at (366.2, -40.5)
- removed the H1 at (459.2, 152.5)
- removed the H1 at (297.0, 151.2)
- removed the H1 at (297.0, -41.8)
- removed the H1 at (229.0, 151.2)
- removed the H1 at (229.0, -41.8)
- removed the H1 at (180.9, -41.0)
- removed the REF** at (-14.3, -63.2)
- removed the REF** at (-14.3, -95.0)
- removed the REF** at (450.7, -63.2)
- removed the REF** at (450.7, -95.0)
- removed SW9: RUNSTOP, RobsFoots:FP-MINITOGLE
- added +12V: LED +12, AA-ROB-FULL:FP-LED_D5.0mm, F.Cu at (141.3, 78.4)
- added +12V: LED +12, AA-ROB-FULL:FP-LED_D5.0mm, F.Cu at (141.3, 128.4)
- added +12V: LED +12, AA-ROB-FULL:FP-LED_D5.0mm, F.Cu at (141.3, 103.4)
- added +12V: LED +12, AA-ROB-FULL:FP-LED_D5.0mm, F.Cu at (141.3, 53.4)
- added +12V: LED +12, AA-ROB-FULL:FP-LED_D5.0mm, F.Cu at (141.3, 28.4)
- added +12V: LED +12, AA-ROB-FULL:FP-LED_D5.0mm, F.Cu at (174.8, -20.2)
- added +12V: LED +12, AA-ROB-FULL:FP-LED_D5.0mm, F.Cu at (141.3, 3.38)
- added H1: MountingHole_Pad, MountingHole:MountingHole_3.2mm_M3_DIN965_Pad, B.Cu at (171.3, 121.4)
- added H1: MountingHole_Pad, MountingHole:MountingHole_3.2mm_M3_DIN965_Pad, B.Cu at (147.3, 121.4)
- added H1: MountingHole_Pad, MountingHole:MountingHole_3.2mm_M3_DIN965_Pad, F.Cu at (140.4, 152.0)
- added H1: MountingHole_Pad, MountingHole:MountingHole_3.2mm_M3_DIN965_Pad, F.Cu at (178.4, 152.0)
- added H1: MountingHole_Pad, MountingHole:MountingHole_3.2mm_M3_DIN965_Pad, F.Cu at (178.4, -41.0)
- added H2: MountingHole_Pad, MountingHole:MountingHole_3.2mm_M3_DIN965_Pad, B.Cu at (171.3, 47.9)
- added H2: MountingHole_Pad, MountingHole:MountingHole_3.2mm_M3_DIN965_Pad, B.Cu at (147.3, 47.9)
- added H2: MountingHole_Pad, MountingHole:MountingHole_3.2mm_M3_DIN965_Pad, B.Cu at (159.3, -4.90)
- added REF**: din_socket, AA-ROB-FULL:din_socket, F.Cu at (159.7, 134.2)
- added REF**: din_socket, AA-ROB-FULL:din_socket, F.Cu at (159.7, 109.2)
- added REF**: din_socket, AA-ROB-FULL:din_socket, F.Cu at (159.7, 84.2)
- added REF**: din_socket, AA-ROB-FULL:din_socket, F.Cu at (159.7, 59.1)
- added REF**: din_socket, AA-ROB-FULL:din_socket, F.Cu at (159.7, 34.1)
- added REF**: din_socket, AA-ROB-FULL:din_socket, F.Cu at (151.6, -16.3)
- moved G*** 238.7 mm to (243.7, 100.6)
- moved G*** 211.0 mm to (217.6, 83.0)
- moved H1 2.50 mm to (140.4, -41.0)
Other:
- board size 485.8 x 320.1 mm -> 50 x 200 mm
- board text added: "CLAYTUNE MidiThru By TwinTurbo V0.0.1"
- board text added: "JLCJLCJLCJLC V0.0.1"
- board text removed: "OFF"
- board text removed: "ON"

Commit message: v0.0.1 pcb routed
Parts:
- moved G*** 135.5 mm to (173.5, -15.3)
- moved G*** 91.0 mm to (170.3, 5.25)
- moved REF** 3.89 mm to (148.2, -14.5), turned to 90 degrees
Other:
- board text added: "CLAYTUNE "Thruman Show" By TwinTurbo"
- board text added: "CLAYTUNE - Thrumanshow V0.0.1 - By TwinTurbo - JLCJLCJLCJLC"
- board text added: "MIDI IN"
- board text added: "Power"
- board text added: "Thru #1"
- board text added: "Thru #2"
- board text added: "Thru #3"
- board text added: "Thru #4"
- board text added: "Thru #5"
- board text removed: "BIG RED BUSS"
- board text removed: "CLAYTUNE - Big Red Buss V0.1.0 - By TwinTurbo - JLCJLCJLCJLC"
- board text removed: "CLAYTUNE Big Red Buss By TwinTurbo"
- board text removed: "CLAYTUNE MidiThru By TwinTurbo V0.0.1"
Changed lines of the file:
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@@
   (general
     (thickness 1.6)
-    (drawings 18)
+    (drawings 24)
     (tracks 0)
     (zones 0)
@@
   )
   (module AA-ROB-FULL:din_socket (layer F.Cu)
-    (at 151.61 -16.34)
-    (fp_text reference REF** (at 0.21 7.23) (layer Dwgs.User)
-      (effects (font (size 1 1) (thickness 0.15)))
-    )
-    (fp_text value din_socket (at 0.21 6.23) (layer F.Fab)
-      (effects (font (size 1 1) (thickness 0.15)))
-    )
-    (fp_text user l (at 2.7 -2.3) (layer F.SilkS)
+    (at 148.18 -14.5 90)
+    (fp_text reference REF** (at 0.21 7.23 90) (layer Dwgs.User)
+      (effects (font (size 1 1) (thickness 0.15)))
+    )
+    (fp_text value din_socket (at 0.21 6.23 90) (layer F.Fab)
+      (effects (font (size 1 1) (thickness 0.15)))
+    )
+    (fp_text user l (at 2.7 -2.3 90) (layer F.SilkS)
       (effects (font (size 1 1) (thickness 0.15)))
     )
@@
     (fp_line (start 0.42 -10.86) (end 16.43 -0.34) (layer Dwgs.User) (width 0.12))
     (fp_line (start 0.66 9.78) (end 16.31 0.61) (layer Dwgs.User) (width 0.12))
-    (pad 3 thru_hole circle (at -11.49 0.03) (size 4 4) (drill 3.5) (layers *.Cu *.Mask))
-    (pad 3 thru_hole circle (at 11.51 0.03) (size 4 4) (drill 3.5) (layers *.Cu *.Mask))
-    (pad 1 thru_hole circle (at 0.01 0.03) (size 16 16) (drill 15) (layers *.Cu *.Mask))
+    (pad 3 thru_hole circle (at -11.49 0.03 90) (size 4 4) (drill 3.5) (layers *.Cu *.Mask))
+    (pad 3 thru_hole circle (at 11.51 0.03 90) (size 4 4) (drill 3.5) (layers *.Cu *.Mask))
+    (pad 1 thru_hole circle (at 0.01 0.03 90) (size 16 16) (drill 15) (layers *.Cu *.Mask))
   )
   (module AA-ROB-FULL:FP-LED_D5.0mm (layer F.Cu)
@@
   )
   (module ROBSLIBRARY:shoebw-cu (layer F.Cu)
-    (at 243.66 100.62)
+    (at 173.46 -15.32)
     (fp_text reference G*** (at 0 0) (layer F.SilkS) hide
       (effects (font (size 1.524 1.524) (thickness 0.3)))
@@
   )
   (module ROBSLIBRARY:GFX1FC (layer F.Cu)
-    (at 217.58 82.95)
+    (at 170.27 5.25)
     (fp_text reference G*** (at -25.43 -2.4) (layer F.SilkS) hide
       (effects (font (size 1.524 1.524) (thickness 0.3)))
@@
       (xy -0.647259 -12.024255) (xy -0.626714 -12.016411)) (layer F.Cu) (width 0.01))
   )
+  (gr_text Power (at 176.04 -25.44) (layer F.SilkS)
+    (effects (font (size 3 2) (thickness 0.5)))
+  )
+  (gr_text "MIDI IN" (at 140.19 12.7 90) (layer F.SilkS)
+    (effects (font (size 3 2) (thickness 0.5)))
+  )
+  (gr_line (start 134.324 21.44) (end 186.77 21.44) (layer F.SilkS) (width 1.5))
+  (gr_line (start 134.324 46.44) (end 186.77 46.44) (layer F.SilkS) (width 1.5))
+  (gr_line (start 134.324 71.44) (end 186.77 71.44) (layer F.SilkS) (width 1.5))
+  (gr_line (start 134.324 96.44) (end 186.77 96.44) (layer F.SilkS) (width 1.5))
+  (gr_line (start 134.324 146.44) (end 186.77 146.44) (layer F.SilkS) (width 1.5))
+  (gr_text "Thru #5" (at 140 138 90) (layer F.SilkS)
+    (effects (font (size 3 2) (thickness 0.5)))
+  )
+  (gr_text "Thru #4" (at 140 113 90) (layer F.SilkS)
+    (effects (font (size 3 2) (thickness 0.5)))
+  )
+  (gr_text "Thru #3" (at 140 88 90) (layer F.SilkS)
+    (effects (font (size 3 2) (thickness 0.5)))
+  )
+  (gr_text "Thru #2" (at 140 63 90) (layer F.SilkS)
+    (effects (font (size 3 2) (thickness 0.5)))
+  )
+  (gr_text "Thru #1" (at 140 38 90) (layer F.SilkS)
+    (effects (font (size 3 2) (thickness 0.5)))
+  )
   (gr_line (start 159.33 -7.97) (end 159.33 163.67) (layer Dwgs.User) (width 0.15))
   (gr_text "JLCJLCJLCJLC   V0.0.1" (at 168.26 -29.28) (layer B.SilkS)
     (effects (font (size 1.5 1.5) (thickness 0.3) italic) (justify mirror))
   )
-  (gr_text "CLAYTUNE\nMidiThru\nBy TwinTurbo \nV0.0.1" (at 200.73 51.13 270) (layer B.SilkS)
+  (gr_text CLAYTUNE (at 159.89 151.72) (layer F.Cu)
+    (effects (font (size 3 3) (thickness 0.3)))
+  )
+  (gr_text "CLAYTUNE - Thrumanshow V0.0.1 - By TwinTurbo   - JLCJLCJLCJLC" (at 181.24 78.88 90) (layer B.SilkS)
     (effects (font (size 1.5 1.5) (thickness 0.3) italic) (justify mirror))
-  )
-  (gr_text CLAYTUNE (at 160.02 145.796) (layer F.Cu)
-    (effects (font (size 3 3) (thickness 0.3)))
-  )
-  (gr_text "CLAYTUNE - Big Red Buss V0.1.0 - By TwinTurbo   - JLCJLCJLCJLC" (at 127 64.008 90) (layer B.Cu)
-    (effects (font (size 1.5 1.5) (thickness 0.3) italic))
   )
   (gr_line (start 184.362 155.462) (end 134.362 155.462) (layer Edge.Cuts) (width 0.05))
@@
     (effects (font (size 4 4) (thickness 0.15)))
   )
-  (gr_line (start 95.754 -16.87) (end 120.89 -16.87) (layer F.SilkS) (width 1.5))
-  (gr_line (start 84.384 116.08) (end 109.52 116.08) (layer F.SilkS) (width 1.5))
-  (gr_line (start 84.674 123.93) (end 109.81 123.93) (layer F.SilkS) (width 1.5))
-  (gr_line (start 93.944 -23.92) (end 119.08 -23.92) (layer F.SilkS) (width 1.5))
-  (gr_line (start 89.69 -29.35) (end 114.86 -29.35) (layer F.SilkS) (width 1.5))
-  (gr_text "CLAYTUNE\nBig Red Buss\nBy TwinTurbo\n " (at 208.2 -8.8) (layer F.SilkS)
+  (gr_line (start 134.324 121.44) (end 186.77 121.44) (layer F.SilkS) (width 1.5))
+  (gr_text "CLAYTUNE\n\"Thruman Show\"\nBy TwinTurbo\n " (at 159.55 -36.04) (layer F.SilkS)
     (effects (font (size 2 2) (thickness 0.5)))
-  )
-  (gr_text "\nBIG\nRED\nBUSS\n\n " (at 212.37 135.39) (layer F.SilkS)
-    (effects (font (size 6 6) (thickness 1)))
   )
   (gr_text "For Kate\nBy \nTwinTurbo" (at 162.34 -36.39) (layer B.SilkS)
@@
     (connect_pads (clearance 0.508))
     (min_thickness 0.254)
-    (fill (arc_segments 32) (thermal_gap 0.508) (thermal_bridge_width 0.508))
+    (fill yes (arc_segments 32) (thermal_gap 0.508) (thermal_bridge_width 0.508))
     (polygon
       (pts
@@
     (connect_pads (clearance 0.508))
     (min_thickness 0.254)
-    (fill (arc_segments 32) (thermal_gap 0.508) (thermal_bridge_width 0.508))
+    (fill yes (arc_segments 32) (thermal_gap 0.508) (thermal_bridge_width 0.508))
     (polygon
       (pts
