File: Front/Panel.kicad_pcb (KiCad board)
At the start: 2 copper layers, 50 x 200 mm, 24 parts

Commit message: FP - LED  V0.0.3
Parts:
- removed the +12V at (141.3, 3.38)
Other:
- board text added: "CLAYTUNE - Thrumanshow V0.0.3 - By TwinTurbo - JLCJLCJLCJLC"
- board text removed: "CLAYTUNE - Thrumanshow V0.0.1 - By TwinTurbo - JLCJLCJLCJLC"
- board text removed: "MIDI IN"
Changed lines of the file:
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@@
   (general
     (thickness 1.6)
-    (drawings 24)
+    (drawings 23)
     (tracks 0)
     (zones 0)
-    (modules 24)
+    (modules 23)
     (nets 2)
   )
   (page A4)
   (layers
-    (0 F.Cu signal)
-    (31 B.Cu signal)
+    (0 F.Cu signal hide)
+    (31 B.Cu signal hide)
     (32 B.Adhes user)
     (33 F.Adhes user)
@@
     )
     (pad 1 thru_hole circle (at 1.27 0) (size 5.4 5.4) (drill 5.2) (layers *.Cu *.Mask))
-  )
-  (module AA-ROB-FULL:FP-LED_D5.0mm (layer F.Cu)
-    (at 141.28 3.38 180)
-    (descr "LED, diameter 5.0mm, 2 pins, http://cdn-reichelt.de/documents/datenblatt/A500/LL-504BC2E-009.pdf")
-    (tags "LED diameter 5.0mm 2 pins")
-    (fp_text reference +12V (at 14.65 0.67 90) (layer F.SilkS)
-      (effects (font (size 1.5 1.5) (thickness 0.2)))
-    )
-    (fp_text value "LED +12" (at 13.61 7.92) (layer F.Fab)
-      (effects (font (size 1 1) (thickness 0.15)))
-    )
-    (fp_line (start 4.5 -3.25) (end -1.95 -3.25) (layer F.CrtYd) (width 0.05))
-    (fp_line (start 4.5 3.25) (end 4.5 -3.25) (layer F.CrtYd) (width 0.05))
-    (fp_line (start -1.95 3.25) (end 4.5 3.25) (layer F.CrtYd) (width 0.05))
-    (fp_line (start -1.95 -3.25) (end -1.95 3.25) (layer F.CrtYd) (width 0.05))
-    (fp_text user %R (at 1.25 0) (layer F.Fab)
-      (effects (font (size 0.8 0.8) (thickness 0.2)))
-    )
-    (pad 1 thru_hole circle (at 1.27 0 180) (size 5.4 5.4) (drill 5.2) (layers *.Cu *.Mask)
-      (net 1 GND))
   )
   (module MountingHole:MountingHole_3.2mm_M3_DIN965_Pad (layer B.Cu)
@@
     (effects (font (size 3 2) (thickness 0.5)))
   )
-  (gr_text "MIDI IN" (at 140.19 12.7 90) (layer F.SilkS)
-    (effects (font (size 3 2) (thickness 0.5)))
-  )
   (gr_line (start 134.324 21.44) (end 186.77 21.44) (layer F.SilkS) (width 1.5))
   (gr_line (start 134.324 46.44) (end 186.77 46.44) (layer F.SilkS) (width 1.5))
@@
     (effects (font (size 3 3) (thickness 0.3)))
   )
-  (gr_text "CLAYTUNE - Thrumanshow V0.0.1 - By TwinTurbo   - JLCJLCJLCJLC" (at 181.24 78.88 90) (layer B.SilkS)
+  (gr_text "CLAYTUNE - Thrumanshow V0.0.3 - By TwinTurbo   - JLCJLCJLCJLC" (at 181.24 78.88 90) (layer B.SilkS)
     (effects (font (size 1.5 1.5) (thickness 0.3) italic) (justify mirror))
   )

Commit message: DOC Version Number Update
Other:
- board text added: "Thruman Show V.0.0.3"
- board text removed: "Big Red Buss- PCB V 0.1.0"
